Commit message: gen3_lite_examples_cpp pkg has been added. In addition, the gravity cancellation node has been created.

File: src/gen3_lite_description/urdf/gen3_lite_macro.xacro (robot description, xacro)
@@ -1,5 +1,5 @@
 <?xml version="1.0"?>
 <robot xmlns:xacro="http://www.ros.org/wiki/xacro">
-  <!-- ================= MACRO PRINCIPAL ================= -->
+  <!-- ================= MAIN MACRO ================= -->
   <xacro:macro name="gen3_lite_arm" params="p ns controllers">
   <!-- WORLD -->
@@ -35,8 +35,8 @@
   <link name="${p}shoulder_link">
     <inertial>
-      <origin xyz="2.477E-05 0.02213531 0.09937686"/>
+      <origin xyz="-2.477E-05 -0.02213531 0.09937686"/>
       <mass value="0.95974404"/>
-      <inertia ixx="0.00165947" ixy="2E-08" ixz="3.6E-07"
-              iyy="0.00140355" iyz="0.00034927" izz="0.00089493"/>
+      <inertia ixx="0.00165947" ixy="-2E-08" ixz="3.6E-07"
+              iyy="0.00140355" iyz="-0.00034927" izz="0.00089493"/>
     </inertial>
     <visual>
@@ -60,12 +60,13 @@
     <axis xyz="0 0 1"/>
     <limit lower="-2.69" upper="2.69" effort="10" velocity="1.6"/>
+    <dynamics damping="0.05" friction="0.2"/>
   </joint>
   <!-- JOINT 2 -->
   <link name="${p}arm_link">
     <inertial>
-      <origin xyz="0.02998299 0.21154808 0.0453031"/>
+      <origin xyz="-0.02998299 0.21154808 0.0453031"/>
       <mass value="1.17756164"/>
-      <inertia ixx="0.01149277" ixy="1E-06" ixz="1.6E-07"
-              iyy="0.00102851" iyz="0.00140765" izz="0.01133492"/>
+      <inertia ixx="0.01149277" ixy="1E-06" ixz="-1.6E-07"
+              iyy="0.00102851" iyz="-0.00140765" izz="0.01133492"/>
     </inertial>
     <visual>
@@ -88,12 +89,13 @@
     <origin xyz="0 -0.03 0.115" rpy="1.5708 0 0"/>
     <axis xyz="0 0 1"/>
-    <limit lower="-2.69" upper="2.69" effort="14" velocity="1.6"/>
+    <limit lower="-2.69" upper="2.69" effort="25" velocity="1.6"/>
+    <dynamics damping="0.5" friction="1.0"/>
   </joint>
   <!-- JOINT 3 -->
   <link name="${p}forearm_link">
     <inertial>
-      <origin xyz="0.0301559 0.09502206 0.0073555"/>
+      <origin xyz="-0.0301559 -0.09502206 -0.0073555"/>
       <mass value="0.59767669"/>
-      <inertia ixx="0.00163256" ixy="7.11E-06" ixz="1.54E-06"
+      <inertia ixx="0.00163256" ixy="-7.11E-06" ixz="-1.54E-06"
               iyy="0.00029798" iyz="9.587E-05" izz="0.00169091"/>
     </inertial>
@@ -116,13 +118,14 @@
     <child link="${p}forearm_link"/>
     <origin xyz="0 0.28 0" rpy="-3.1416 0 0"/>
-    <axis xyz="0 0 1"/>
-    <limit lower="-2.69" upper="2.69" effort="10" velocity="1.6"/>
+    <axis xyz="0 0 -1"/>
+    <limit lower="-2" upper="2" effort="10" velocity="1.6"/>
+    <dynamics damping="0.05" friction="0.2"/>
   </joint>
   <!-- WRIST -->
   <link name="${p}lower_wrist_link">
     <inertial>
-      <origin xyz="0.00575149 0.01000443 0.08719207" rpy="0 0 0" />
+      <origin xyz="0.00575149 -0.01000443 0.08719207" rpy="0 0 0" />
       <mass value="0.52693412" />
-      <inertia ixx="0.00069098" ixy="2.4E-07" ixz="0.00016483" iyy="0.00078519" iyz="7.4E-07" izz="0.00034115" />
+      <inertia ixx="0.00069098" ixy="-2.4E-07" ixz="0.00016483" iyy="0.00078519" iyz="7.4E-07" izz="0.00034115" />
     </inertial>
     <visual>
@@ -146,10 +149,11 @@
     <axis xyz="0 0 1"/>
     <limit lower="-2.59" upper="2.59" effort="7" velocity="1.6"/>
+    <dynamics damping="0.05" friction="0.2"/>
   </joint>
   <link name="${p}upper_wrist_link">
     <inertial>
-      <origin xyz="0.08056517 0.00980409 0.01872799" rpy="0 0 0" />
+      <origin xyz="-0.08056517 -0.00980409 0.01872799" rpy="0 0 0" />
       <mass value="0.58097325" />
-      <inertia ixx="0.00021268" ixy="5.21E-06" ixz="2.91E-06" iyy="0.00106371" iyz="1.1E-07" izz="0.00108465" />
+      <inertia ixx="0.00021268" ixy="5.21E-06" ixz="-2.91E-06" iyy="0.00106371" iyz="1.1E-07" izz="0.00108465" />
     </inertial>
     <visual>
@@ -173,4 +177,5 @@
     <axis xyz="0 0 1"/>
     <limit lower="-2.57" upper="2.57" effort="7" velocity="1.6"/>
+    <dynamics damping="0.05" friction="0.2"/>
   </joint>
       <!-- JOINT 6 CONECTADO DIRECTO AL GRIPPER -->
@@ -181,4 +186,5 @@
     <axis xyz="0 0 1"/>
     <limit lower="-2.59" upper="2.59" effort="7" velocity="3.2"/>
+    <dynamics damping="0.05" friction="0.2"/>
   </joint>
   <!-- ================= GRIPPER ================= -->
@@ -226,5 +232,5 @@
     </collision>
   </link>
-  <joint name="${p}right_finger_bottom_joint" type="revolute">
+  <joint name="${p}right_finger_bottom_joint" type="fixed">
     <origin xyz="0 -0.030501 0.070003" rpy="0 1.5708 0"/>
     <parent link="${p}gripper_base_link"/>
@@ -255,5 +261,5 @@
     </collision>
   </link>
-  <joint name="${p}right_finger_tip_joint" type="revolute">
+  <joint name="${p}right_finger_tip_joint" type="fixed">
     <origin xyz="-0.045636 0.020423 0"/>
     <parent link="${p}right_finger_prox_link"/>
@@ -285,5 +291,5 @@
     </collision>
   </link>
-  <joint name="${p}left_finger_bottom_joint" type="revolute">
+  <joint name="${p}left_finger_bottom_joint" type="fixed">
     <origin xyz="0 0.0305 0.070003" rpy="0 1.5708 0"/>
     <parent link="${p}gripper_base_link"/>
@@ -315,5 +321,5 @@
     </collision>
   </link>
-  <joint name="${p}left_finger_tip_joint" type="revolute">
+  <joint name="${p}left_finger_tip_joint" type="fixed">
     <origin xyz="-0.045636 -0.020423 6.9901E-05"/>
     <parent link="${p}left_finger_prox_link"/>
